File: motorDriver/motorDriver.kicad_pcb (KiCad board)
At the start: 2 copper layers, 29.5 x 28.7 mm, 179 parts, among them P1 CONN_01X03, P2 Input, P3 Output, U1 TB6593FNG

Commit message: Removed some stitch vias from near other footprints
Parts:
- removed REF**111111101, REF**11111191: Via, GoGoGo:Via
Changed lines of the file:
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@@
 (kicad_pcb (version 4) (host pcbnew 0.201508140901+6091~28~ubuntu14.04.1-product)
   (general
-    (links 201)
+    (links 199)
     (no_connects 0)
     (area 137.108028 72.9361 176.423401 106.08056)
@@
     (tracks 116)
     (zones 0)
-    (modules 179)
+    (modules 177)
     (nets 15)
   )
@@
       (effects (font (size 1 1) (thickness 0.15)))
     )
-    (fp_text value Via (at 0 1.27) (layer F.Fab) hide
-      (effects (font (size 1 1) (thickness 0.15)))
-    )
-    (pad 1 thru_hole circle (at 0 0) (size 0.6858 0.6858) (drill 0.3302) (layers *.Cu *.Mask F.SilkS)
-      (net 1 GND) (zone_connect 2))
-  )
-  (module GoGoGo:Via (layer F.Cu)
-    (at 155.194 94.996)
-    (fp_text reference REF**111111101 (at 0 -1.27) (layer F.SilkS) hide
-      (effects (font (size 1 1) (thickness 0.15)))
-    )
-    (fp_text value Via (at 0 1.27) (layer F.Fab) hide
-      (effects (font (size 1 1) (thickness 0.15)))
-    )
-    (pad 1 thru_hole circle (at 0 0) (size 0.6858 0.6858) (drill 0.3302) (layers *.Cu *.Mask F.SilkS)
-      (net 1 GND) (zone_connect 2))
-  )
-  (module GoGoGo:Via (layer F.Cu)
-    (at 153.924 94.996)
-    (fp_text reference REF**11111191 (at 0 -1.27) (layer F.SilkS) hide
-      (effects (font (size 1 1) (thickness 0.15)))
-    )
