File: MotorEncoderBoardBO/MotorEncoderBoard.kicad_pcb (KiCad board)
At the start: 2 copper layers, 24.3 x 28.1 mm, 13 parts, among them P1 PWR, P2 Out, U1 RPI-579N1, U2 LM311D

Commit message: Enhanced the board with indicator LEDs
Parts:
- added D1: Led_Small, LEDs:LED_0805, F.Cu at (159.5, 88.0)
- added R6: 470, Resistors_SMD:R_0805_HandSoldering, F.Cu at (159.0, 90.4)
- P2: value Out -> CONN_01X03; footprint Pin_Headers:Pin_Header_Straight_1x02 -> Pin_Headers:Pin_Header_Straight_1x03
- moved R3 7.90 mm to (163.4, 83.9), turned to 180 degrees
- moved C1 1.15 mm to (155.1, 87.5)
- moved R1 0.25 mm to (154.9, 96.8)
- moved P2 0.18 mm to (151.0, 96.1)
Connections:
- P2 pad 2: GND -> /Output
Routing:
- net /Output: track 6.81 -> 24.4 mm
- net Net-(R3-Pad1): track 13.9 -> 3.48 mm
- net Net-(D1-Pad1): track 0.00 -> 2.50 mm
- net VCC: track 17.5 -> 18.9 mm
Other:
- board text added: "GND Out TP2"
- board text added: "GND Vcc"
- board text removed: "Out"
- board text removed: "Vcc"
